File: ControlsSim.kicad_sch (KiCad schematic)
At the start: 26 parts, among them J2 Accelerator Pot, J3 Brake Button, J5 Motor Contactors, J6 Array Contactors, J7 Rotary Switch, SW2 SW_Rotary2x6

Commit message: Updated version history and implemented a fix for 3dmodels to be applied next commit
Parts:
- S1: footprint Footprints:TS16121295BK260SMTTR -> TS16121295BK260SMTTR
Other:
- note added: "Future Changes:"
Changed lines of the file:
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@@
+    (stroke (width 0) (type default))
+  )
+  (polyline (pts (xy 187.96 34.29) (xy 187.96 113.03))
     (stroke (width 0) (type default))
   )
@@
     (stroke (width 0) (type default))
   )
+  (polyline (pts (xy 187.96 34.29) (xy 265.43 34.29))
+    (stroke (width 0) (type default))
+  )
   (wire (pts (xy 64.77 78.105) (xy 71.12 78.105))
     (stroke (width 0) (type default))
@@
     (stroke (width 0) (type default))
   )
+  (polyline (pts (xy 265.43 113.03) (xy 187.96 113.03))
+    (stroke (width 0) (type default))
+  )
   (wire (pts (xy 71.12 131.445) (xy 71.12 133.35))
     (stroke (width 0) (type default))
@@
   )
   (wire (pts (xy 167.005 71.12) (xy 164.465 71.12))
+    (stroke (width 0) (type default))
+  )
+  (polyline (pts (xy 265.43 34.29) (xy 265.43 113.03))
     (stroke (width 0) (type default))
   )
@@
     (effects (font (size 1.27 1.27)) (justify left bottom))
   )
+  (text "Future Changes:" (at 196.85 64.77 0)
+    (effects (font (size 1.27 1.27)) (justify left bottom))
+  )
   (text "EL3H7 is operating at forward current ~20mA" (at 85.09 40.005 0)
     (effects (font (size 1.27 1.27)) (justify left bottom))
@@
       (effects (font (size 1.27 1.27)) hide)
     )
-    (property "Datasheet" "" (at 51.435 73.025 0)
+    (property "Datasheet" "https://www.mouser.com/ProductDetail/Kingbright/APTD2012LVBC-D?qs=AQlKX63v8RtBBvAHcuxu8A%3D%3D" (at 51.435 73.025 0)
       (effects (font (size 1.27 1.27)) hide)
     )
@@
       (effects (font (size 1.27 1.27)) hide)
     )
-    (property "Datasheet" "~" (at 65.405 150.495 0)
+    (property "Datasheet" "https://www.mouser.com/ProductDetail/71-CRCW080510K0FKEAC" (at 65.405 150.495 0)
       (effects (font (size 1.27 1.27)) hide)
     )
@@
       (effects (font (size 1.27 1.27)) hide)
     )
-    (property "Datasheet" "" (at 51.435 78.105 0)
+    (property "Datasheet" "https://www.mouser.com/ProductDetail/604-APTD2012LCGCK" (at 51.435 78.105 0)
       (effects (font (size 1.27 1.27)) hide)
     )
@@
       (effects (font (size 1.27 1.27)) hide)
     )
-    (property "Datasheet" "~" (at 76.2 127.635 0)
+    (property "Datasheet" "https://tools.molex.com/pdm_docs/ps/PS-43045.pdf" (at 76.2 127.635 0)
       (effects (font (size 1.27 1.27)) hide)
     )
@@
       (effects (font (size 1.27 1.27)) hide)
     )
-    (property "Datasheet" "~" (at 62.23 78.105 0)
+    (property "Datasheet" "https://www.mouser.com/ProductDetail/Vishay-Dale/CRCW0805330RJNEAC?qs=sGAEpiMZZMvdGkrng054t0DrEhLhGh8gFaieh3KXECz0vzyY6hoijA%3D%3D" (at 62.23 78.105 0)
       (effects (font (size 1.27 1.27)) hide)
     )
@@
       (effects (font (size 1.27 1.27)) hide)
     )
-    (property "Datasheet" "" (at 64.135 52.07 0)
+    (property "Datasheet" "https://www.mouser.com/ProductDetail/Vishay-Dale/CRCW0805330RJNEAC?qs=sGAEpiMZZMvdGkrng054t0DrEhLhGh8gFaieh3KXECz0vzyY6hoijA%3D%3D" (at 64.135 52.07 0)
       (effects (font (size 1.27 1.27)) hide)
     )
@@
       (effects (font (size 1.27 1.27)) hide)
     )
-    (property "Datasheet" "~" (at 73.66 78.105 0)
+    (property "Datasheet" "https://www.mouser.com/ProductDetail/Vishay-Dale/CRCW0805330RJNEAC?qs=sGAEpiMZZMvdGkrng054t0DrEhLhGh8gFaieh3KXECz0vzyY6hoijA%3D%3D" (at 73.66 78.105 0)
       (effects (font (size 1.27 1.27)) hide)
     )
@@
       (effects (font (size 1.27 1.27)))
     )
-    (property "Footprint" "Footprints:TS16121295BK260SMTTR" (at 50.8 145.415 0)
+    (property "Footprint" "TS16121295BK260SMTTR" (at 50.8 145.415 0)
       (effects (font (size 1.27 1.27)) (justify left) hide)
     )
@@
       (effects (font (size 1.27 1.27)) hide)
     )
-    (property "Datasheet" "" (at 73.66 52.07 0)
+    (property "Datasheet" "https://www.mouser.com/ProductDetail/Vishay-Dale/CRCW0805330RJNEAC?qs=sGAEpiMZZMvdGkrng054t0DrEhLhGh8gFaieh3KXECz0vzyY6hoijA%3D%3D" (at 73.66 52.07 0)
       (effects (font (size 1.27 1.27)) hide)
     )
@@
       (effects (font (size 1.27 1.27)) hide)
     )
-    (property "Datasheet" "~" (at 76.2 147.955 0)
+    (property "Datasheet" "https://tools.molex.com/pdm_docs/ps/PS-43045.pdf" (at 76.2 147.955 0)
       (effects (font (size 1.27 1.27)) hide)
     )
@@
       (effects (font (size 1.27 1.27)) hide)
     )
-    (property "Datasheet" "" (at 64.135 46.99 0)
+    (property "Datasheet" "https://www.mouser.com/ProductDetail/Vishay-Dale/CRCW0805330RJNEAC?qs=sGAEpiMZZMvdGkrng054t0DrEhLhGh8gFaieh3KXECz0vzyY6hoijA%3D%3D" (at 64.135 46.99 0)
       (effects (font (size 1.27 1.27)) hide)
     )
@@
       (effects (font (size 1.27 1.27)) hide)
     )
-    (property "Datasheet" "" (at 73.66 46.99 0)
+    (property "Datasheet" "https://www.mouser.com/ProductDetail/Vishay-Dale/CRCW0805330RJNEAC?qs=sGAEpiMZZMvdGkrng054t0DrEhLhGh8gFaieh3KXECz0vzyY6hoijA%3D%3D" (at 73.66 46.99 0)
       (effects (font (size 1.27 1.27)) hide)
     )
@@
       (effects (font (size 1.27 1.27)) hide)
     )
-    (property "Datasheet" "~" (at 88.265 49.53 0)
+    (property "Datasheet" "https://tools.molex.com/pdm_docs/ps/PS-43650.pdf" (at 88.265 49.53 0)
       (effects (font (size 1.27 1.27)) hide)
     )
@@
       (effects (font (size 1.27 1.27)) hide)
     )
-    (property "Datasheet" "~" (at 67.945 73.025 0)
+    (property "Datasheet" "https://www.mouser.com/ProductDetail/Vishay-Dale/CRCW0805330RJNEAC?qs=sGAEpiMZZMvdGkrng054t0DrEhLhGh8gFaieh3KXECz0vzyY6hoijA%3D%3D" (at 67.945 73.025 0)
       (effects (font (size 1.27 1.27)) hide)
     )
@@
       (effects (font (size 1.27 1.27)) hide)
     )
-    (property "Datasheet" "~" (at 88.265 75.565 0)
+    (property "Datasheet" "https://tools.molex.com/pdm_docs/ps/PS-43650.pdf" (at 88.265 75.565 0)
       (effects (font (size 1.27 1.27)) hide)
     )
@@
       (effects (font (size 1.27 1.27)) hide)
     )
-    (property "Datasheet" "~" (at 118.11 81.28 0)
+    (property "Datasheet" "https://tools.molex.com/pdm_docs/ps/PS-43045.pdf" (at 118.11 81.28 0)
       (effects (font (size 1.27 1.27)) hide)
     )
@@
       (effects (font (size 1.27 1.27)) hide)
     )
-    (property "Datasheet" "" (at 51.435 52.07 0)
-      (effects (font (size 1.27 1.27)) hide)
-    )
+    (property "Datasheet" "https://www.mouser.com/ProductDetail/604-APTD2012LSURCK" (at 51.435 52.07 0)
+      (effects (font (size 1.27 1.27)) hide)
+    )
